File: hardware/kv5x_devboard.kicad_pcb (KiCad board)
At the start: 2 copper layers, 5 parts, among them J1 JTAG/SWD Connector, U1 MKV56F1M0VLL24

Commit message: USB interface half done
Parts:
- added C10: 15pF, Capacitor_SMD:C_0402_1005Metric, F.Cu at (113.5, 105.5)
- added C11: 15pF, Capacitor_SMD:C_0402_1005Metric, F.Cu at (110.0, 108.5)
- added C12: 1uF, Capacitor_SMD:C_0402_1005Metric, F.Cu at (69.0, 109.0)
- added C13: 0.1uF, Capacitor_SMD:C_0402_1005Metric, F.Cu at (110.5, 98.5)
- added C14: 0.1uF, Capacitor_SMD:C_0402_1005Metric, F.Cu at (93.0, 100.0)
- added C15: 0.1uF, Capacitor_SMD:C_0402_1005Metric, F.Cu at (93.0, 95.5)
- added C16: 0.1uF, Capacitor_SMD:C_0402_1005Metric, F.Cu at (102.0, 105.0)
- added FB1: 330R, Resistor_SMD:R_0603_1608Metric, F.Cu at (70.3, 87.0)
- added FB2: 330R, Resistor_SMD:R_0603_1608Metric, F.Cu at (69.0, 106.5)
- added J2: USB_C_Receptacle_USB2.0_16P, Connector_USB:USB_C_Receptacle_Palconn_UTC16-G, F.Cu at (70.7, 95.7)
- added R10: 1M, Resistor_SMD:R_0402_1005Metric, F.Cu at (106.0, 102.5)
- added R4: 4.7k, Resistor_SMD:R_0402_1005Metric, F.Cu at (114.5, 97.5)
- added R5: 10k, Resistor_SMD:R_0402_1005Metric, F.Cu at (114.5, 100.0)
- added R6: 33R, Resistor_SMD:R_0402_1005Metric, F.Cu at (86.5, 94.5)
- added R7: 33R, Resistor_SMD:R_0402_1005Metric, F.Cu at (86.5, 96.5)
- added R8: 5.1k, Resistor_SMD:R_0402_1005Metric, F.Cu at (79.5, 94.0)
- added R9: 5.1k, Resistor_SMD:R_0402_1005Metric, F.Cu at (79.5, 96.5)
- added TP1: TestPoint, 0_kv5x_devboard:TestPoint_Pad_D0.5mm, F.Cu at (96.0, 108.0)
- added TP2: TestPoint, 0_kv5x_devboard:TestPoint_Pad_D0.5mm, F.Cu at (98.5, 108.0)
- added TP3: TestPoint, 0_kv5x_devboard:TestPoint_Pad_D0.5mm, F.Cu at (116.5, 97.5)
- added TP4: TestPoint, 0_kv5x_devboard:TestPoint_Pad_D0.5mm, F.Cu at (72.0, 106.0)
- added U2: MK20DX128VLF5, 0_kv5x_devboard:MK20DX128VLF5, F.Cu at (100.0, 98.0)
- added Y1: ECS-80-12-33-JGN-TR, Crystal:Crystal_SMD_3225-4Pin_3.2x2.5mm, F.Cu at (110.0, 105.5)
- moved J1 18.1 mm to (127.0, 133.0)
- moved R1 18.1 mm to (137.8, 130.0)
- moved R2 18.1 mm to (137.8, 132.5)
- moved R3 18.1 mm to (137.8, 135.0)
