File: hardware/sch/usb_interface.kicad_sch (KiCad schematic)
At the start: 0 parts

Commit message: USB interface half done
Parts:
- added C10, C11: 15pF, Capacitor_SMD:C_0402_1005Metric, symbol Device:C
- added C12: 1uF, Capacitor_SMD:C_0402_1005Metric, symbol Device:C
- added C13, C14, C15, C16: 0.1uF, Capacitor_SMD:C_0402_1005Metric, symbol Device:C
- added FB1, FB2: 330R, Resistor_SMD:R_0603_1608Metric, symbol Device:FerriteBead
- added J2: USB_C_Receptacle_USB2.0_16P, Connector_USB:USB_C_Receptacle_Palconn_UTC16-G, symbol Connector:USB_C_Receptacle_USB2.0_16P
- added R10: 1M, Resistor_SMD:R_0402_1005Metric, symbol Device:R
- added R4: 4.7k, Resistor_SMD:R_0402_1005Metric, symbol Device:R
- added R5: 10k, Resistor_SMD:R_0402_1005Metric, symbol Device:R
- added R6, R7: 33R, Resistor_SMD:R_0402_1005Metric, symbol Device:R
- added R8, R9: 5.1k, Resistor_SMD:R_0402_1005Metric, symbol Device:R
- added TP1, TP2, TP3, TP4: TestPoint, 0_kv5x_devboard:TestPoint_Pad_D0.5mm, symbol 0_kv5x_devboard:TestPoint_0.5mm
- added U2: MK20DX128VLF5, 0_kv5x_devboard:MK20DX128VLF5, symbol 0_kv5x_devboard:MK20DX128VLF5
- added Y1: ECS-80-12-33-JGN-TR, Crystal:Crystal_SMD_3225-4Pin_3.2x2.5mm, symbol Device:Crystal_GND24
Connections:
- new net: J2.A5 (CC1), R8.1
- new net: J2.B5 (CC2), R9.1
- new net +3.3V: C14.1, C15.1, C16.1, U2.1 (VDD1), U2.10 (VREFH), U2.16 (VBAT), U2.22 (VDD2), U2.6 (VREGIN), U2.9 (VDDA)
- new net GND: C10.2, C11.2, C12.2, C13.2, C14.2, C15.2, C16.2, FB1.2, J2.A1 (GND), J2.A12 (GND), J2.B1 (GND), J2.B12 (GND), R5.2, R8.2, R9.2, U2.11 (VREFL), U2.12 (VSSA), U2.2 (VSS1), U2.23 (VSS2), Y1.2, Y1.4
- new net K20_JTAG_TCLK: U2.17 (JTAG_TCLK/SWD_CLK/EZP_CLK/TSI0_CH1/PTA0/*UART0_CTS/*UART0_COL/FTM0_CH5)
- new net K20_JTAG_TDI: U2.18 (JTAG_TDI/EZP_DI/TSI0_CH2/PTA1/UART0_RX/FTM0_CH6)
- new net K20_JTAG_TDO: U2.19 (JTAG_TDO/TRACE_SWO/EZP_DO/TSI0_CH3/PTA2/UART0_TX/FTM0_CH7)
- new net K20_JTAG_TMS: U2.20 (JTAG_TMS/SWD_DIO/TSI0_CH4/PTA3/*UART0_RTS/FTM0_CH0)
- new net SDA_USB_DM: R7.2, U2.4 (USB0_DM)
- new net SDA_USB_DP: R6.2, U2.3 (USB0_DP)
- new net SDA_XTAL_IN: C11.1, R10.2, U2.24 (EXTAL0/PTA18/FTM0_FLT2/FTM_CLKIN0), Y1.1
- new net SDA_XTAL_OUT: C10.1, R10.1, U2.25 (XTAL0/PTA19/FTM1_FLT0/FTM_CLKIN1/LPTMR0_ALT1), Y1.3
- new net SDA_~{RESET}: C13.1, R4.2, R5.1, TP3.1, U2.26 (~{RESET})
- new net TC_EXTAL_TP: TP1.1, U2.15 (EXTAL32)
- new net TC_XTAL_TP: TP2.1, U2.14 (XTAL32)
- new net USB_D+: J2.A6 (D+), J2.B6 (D+), R6.1
- new net USB_D-: J2.A7 (D-), J2.B7 (D-), R7.1
- new net USB_SHIELD: FB1.1, J2.S1 (SHIELD)
- new net USB_VBUS: FB2.1, J2.A4 (VBUS), J2.A9 (VBUS), J2.B4 (VBUS), J2.B9 (VBUS)
- new net VBUS: C12.1, FB2.2, R4.1, TP4.1
- no-connect marks 0 -> 6
Other:
- note added: "TODO: - RESET circuit (See reference design) - K20 to KV5x connections (SWDIO, SCLK, UART) (See reference design) - SDA LED indicator (See reference design) - Find a use for the other K20 pins"
